File: hardware/macropad.kicad_pcb (KiCad board)
At the start: 2 copper layers, 63.5 x 106.7 mm, 27 parts, among them J2 Conn_01x06, J3 I2C Screen, J4 SPI Screen, SW1 SW_Push, SW10 SW_Push, SW2 SW_Push, SW3 SW_Push, SW4 SW_Push, SW5 SW_Push, SW6 SW_Push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

Commit message: :construction: First draft front panel
Parts:
- added H1: MountingHole, MountingHole:MountingHole_3.2mm_M3, F.Cu at (168.0, 26.8)
- added H2: MountingHole, MountingHole:MountingHole_3.2mm_M3, F.Cu at (225.1, 26.8)
- added H3: MountingHole, MountingHole:MountingHole_3.2mm_M3, F.Cu at (168.0, 127.2)
- added H4: MountingHole, MountingHole:MountingHole_3.2mm_M3, F.Cu at (225.1, 127.2)
Other:
- board size 63.5 x 106.7 mm -> 164.8 x 106.9 mm
Changed lines of the file:
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@@
   (net 41 "ROW0")
   (net 42 "COL0")
+  (footprint "MountingHole:MountingHole_3.2mm_M3" (layer "F.Cu")
+    (at 167.964101 26.845)
+    (descr "Mounting Hole 3.2mm, no annular, M3")
+    (tags "mounting hole 3.2mm no annular m3")
+    (property "Sheetfile" "macropad.kicad_sch")
+    (property "Sheetname" "")
+    (attr exclude_from_pos_files)
+    (fp_text reference "H1" (at 0 -4.2) (layer "F.SilkS") hide
+      (effects (font (size 1 1) (thickness 0.15)))
+    )
+    (fp_text value "MountingHole" (at 0 4.2) (layer "F.Fab")
+      (effects (font (size 1 1) (thickness 0.15)))
+    )
+    (fp_text user "${REFERENCE}" (at 0 0) (layer "F.Fab")
+      (effects (font (size 1 1) (thickness 0.15)))
+    )
+    (fp_circle (center 0 0) (end 3.2 0) (layer "Cmts.User") (width 0.15) (fill none))
+    (fp_circle (center 0 0) (end 3.45 0) (layer "F.CrtYd") (width 0.05) (fill none))
+    (pad "" np_thru_hole circle (at 0 0) (size 3.2 3.2) (drill 3.2) (layers *.Cu *.Mask))
+  )
+  (footprint "MountingHole:MountingHole_3.2mm_M3" (layer "F.Cu")
+    (at 167.964101 127.175)
+    (descr "Mounting Hole 3.2mm, no annular, M3")
+    (tags "mounting hole 3.2mm no annular m3")
+    (property "Sheetfile" "macropad.kicad_sch")
+    (property "Sheetname" "")
+    (attr exclude_from_pos_files)
+    (fp_text reference "H3" (at 0 -4.2) (layer "F.SilkS") hide
+      (effects (font (size 1 1) (thickness 0.15)))
+    )
+    (fp_text value "MountingHole" (at 0 4.2) (layer "F.Fab")
+      (effects (font (size 1 1) (thickness 0.15)))
+    )
+    (fp_text user "${REFERENCE}" (at 0 0) (layer "F.Fab")
+      (effects (font (size 1 1) (thickness 0.15)))
+    )
+    (fp_circle (center 0 0) (end 3.2 0) (layer "Cmts.User") (width 0.15) (fill none))
+    (fp_circle (center 0 0) (end 3.45 0) (layer "F.CrtYd") (width 0.05) (fill none))
+    (pad "" np_thru_hole circle (at 0 0) (size 3.2 3.2) (drill 3.2) (layers *.Cu *.Mask))
+  )
   (footprint "Switch_Keyboard_Hotswap_Kailh:SW_Hotswap_Kailh_MX" (layer "F.Cu")
     (at 76.2 76.2)
@@
   )
   (footprint "MountingHole:MountingHole_3.2mm_M3" (layer "F.Cu")
+    (at 225.114101 26.845)
+    (descr "Mounting Hole 3.2mm, no annular, M3")
+    (tags "mounting hole 3.2mm no annular m3")
+    (property "Sheetfile" "macropad.kicad_sch")
+    (property "Sheetname" "")
+    (attr exclude_from_pos_files)
+    (fp_text reference "H2" (at 0 -4.2) (layer "F.SilkS") hide
+      (effects (font (size 1 1) (thickness 0.15)))
+    )
+    (fp_text value "MountingHole" (at -54.61 4.2) (layer "B.Fab")
+      (effects (font (size 1 1) (thickness 0.15)) (justify mirror))
+    )
+    (fp_text user "${REFERENCE}" (at 0 0) (layer "F.Fab")
+      (effects (font (size 1 1) (thickness 0.15)))
+    )
+    (fp_circle (center 0 0) (end 3.2 0) (layer "Cmts.User") (width 0.15) (fill none))
+    (fp_circle (center 0 0) (end 3.45 0) (layer "F.CrtYd") (width 0.05) (fill none))
+    (pad "" np_thru_hole circle (at 0 0) (size 3.2 3.2) (drill 3.2) (layers *.Cu *.Mask))
+  )
+  (footprint "MountingHole:MountingHole_3.2mm_M3" (layer "F.Cu")
     (at 66.675 127)
     (descr "Mounting Hole 3.2mm, no annular, M3")
@@
     (fp_text value "MountingHole" (at -54.61 4.2) (layer "B.Fab")
       (effects (font (size 1 1) (thickness 0.15)) (justify mirror))
+    )
+    (fp_text user "${REFERENCE}" (at 0 0) (layer "F.Fab")
+      (effects (font (size 1 1) (thickness 0.15)))
+    )
+    (fp_circle (center 0 0) (end 3.2 0) (layer "Cmts.User") (width 0.15) (fill none))
+    (fp_circle (center 0 0) (end 3.45 0) (layer "F.CrtYd") (width 0.05) (fill none))
+    (pad "" np_thru_hole circle (at 0 0) (size 3.2 3.2) (drill 3.2) (layers *.Cu *.Mask))
+  )
+  (footprint "MountingHole:MountingHole_3.2mm_M3" (layer "F.Cu")
+    (at 225.114101 127.175)
+    (descr "Mounting Hole 3.2mm, no annular, M3")
+    (tags "mounting hole 3.2mm no annular m3")
+    (property "Sheetfile" "macropad.kicad_sch")
+    (property "Sheetname" "")
+    (attr exclude_from_pos_files)
+    (fp_text reference "H4" (at 0 -4.2) (layer "F.SilkS") hide
+      (effects (font (size 1 1) (thickness 0.15)))
+    )
+    (fp_text value "MountingHole" (at 0 4.2) (layer "F.Fab")
+      (effects (font (size 1 1) (thickness 0.15)))
     )
     (fp_text user "${REFERENCE}" (at 0 0) (layer "F.Fab")
@@
     )
   )
+  (gr_rect (start 170.489101 107.475) (end 184.489101 121.475) (layer "Edge.Cuts") (width 0.1) (fill none))
   (gr_line (start 127 49.5) (end 127 130.175) (layer "Edge.Cuts") (width 0.1))
+  (gr_rect (start 208.589101 69.375) (end 222.589101 83.375) (layer "Edge.Cuts") (width 0.1) (fill none))
   (gr_line (start 63.5 23.495) (end 127 23.495) (layer "Edge.Cuts") (width 0.1))
+  (gr_line (start 164.789101 130.35) (end 228.289101 130.35) (layer "Edge.Cuts") (width 0.1))
+  (gr_rect (start 170.489101 69.375) (end 184.489101 83.375) (layer "Edge.Cuts") (width 0.1) (fill none))
+  (gr_rect (start 170.489101 88.425) (end 184.489101 102.425) (layer "Edge.Cuts") (width 0.1) (fill none))
   (gr_line (start 127 37) (end 127 23.495) (layer "Edge.Cuts") (width 0.1))
+  (gr_rect (start 189.539101 88.425) (end 203.539101 102.425) (layer "Edge.Cuts") (width 0.1) (fill none))
+  (gr_line (start 164.789101 23.67) (end 164.789101 130.35) (layer "Edge.Cuts") (width 0.1))
   (gr_line (start 63.5 130.175) (end 127 130.175) (layer "Edge.Cuts") (width 0.1))
   (gr_line (start 125.75 48.25) (end 120.5 48.25) (layer "Edge.Cuts") (width 0.1))
+  (gr_line (start 164.789101 23.67) (end 228.289101 23.67) (layer "Edge.Cuts") (width 0.1))
   (gr_arc (start 120.5 48.25) (mid 119.616117 47.883883) (end 119.25 47) (layer "Edge.Cuts") (width 0.1))
+  (gr_rect (start 208.589101 50.325) (end 222.589101 64.325) (layer "Edge.Cuts") (width 0.1) (fill none))
   (gr_arc (start 125.75 48.25) (mid 126.633883 48.616117) (end 127 49.5) (layer "Edge.Cuts") (width 0.1))
   (gr_line (start 125.75 38.25) (end 120.5 38.25) (layer "Edge.Cuts") (width 0.1))
+  (gr_rect (start 170.649101 30.98) (end 204.649101 56.98) (layer "Edge.Cuts") (width 0.1) (fill none))
+  (gr_rect (start 189.539101 69.375) (end 203.539101 83.375) (layer "Edge.Cuts") (width 0.1) (fill none))
   (gr_arc (start 119.25 39.5) (mid 119.616117 38.616117) (end 120.5 38.25) (layer "Edge.Cuts") (width 0.1))
   (gr_line (start 119.25 47) (end 119.25 39.5) (layer "Edge.Cuts") (width 0.1))
   (gr_line (start 63.5 23.495) (end 63.5 130.175) (layer "Edge.Cuts") (width 0.1))
+  (gr_line (start 228.289101 130.35) (end 228.289101 23.67) (layer "Edge.Cuts") (width 0.1))
   (gr_arc (start 127 37) (mid 126.633883 37.883883) (end 125.75 38.25) (layer "Edge.Cuts") (width 0.1))
+  (gr_rect (start 208.589101 88.425) (end 222.589101 102.425) (layer "Edge.Cuts") (width 0.1) (fill none))
+  (gr_rect (start 208.589101 107.475) (end 222.589101 121.475) (layer "Edge.Cuts") (width 0.1) (fill none))
+  (gr_rect (start 189.539101 107.475) (end 203.539101 121.475) (layer "Edge.Cuts") (width 0.1) (fill none))
   (gr_text "<-  USB THIS WAY" (at 110.5 43) (layer "B.SilkS")
     (effects (font (size 1 1) (thickness 0.15)) (justify mirror))
@@
       (effects (font (size 1.5 1.5) (thickness 0.3)))
     )
+    (format (units 3) (units_format 1) (precision 4))
+    (style (thickness 0.2) (arrow_length 1.27) (text_position_mode 0) (extension_height 0.58642) (extension_offset 0.5) keep_text_aligned)
+  )
+  (dimension (type aligned) (layer "User.1")
+    (pts (xy 167.964101 127.175) (xy 225.114101 127.175))
+    (height 25.4)
+    (gr_text "57,1500 mm" (at 196.539101 150.775) (layer "User.1")
+      (effects (font (size 1.5 1.5) (thickness 0.3)))
+    )
+    (format (units 3) (units_format 1) (precision 4))
+    (style (thickness 0.2) (arrow_length 1.27) (text_position_mode 0) (extension_height 0.58642) (extension_offset 0.5) keep_text_aligned)
+  )
+  (dimension (type aligned) (layer "User.1")
+    (pts (xy 164.789101 130.35) (xy 228.289101 130.35))
+    (height 29.845)
+    (gr_text "63,5000 mm" (at 196.539101 158.395) (layer "User.1")
+      (effects (font (size 1.5 1.5) (thickness 0.3)))
+    )
